Commit message: replace collision meshes with boxes

File: pal_wsg_gripper_description/urdf/gripper.urdf.xacro (robot description, xacro)
@@ -57,7 +57,9 @@
       </visual>
       <collision>
-        <origin xyz="0 0 0" rpy="0 0 0" />
+        <!-- <origin xyz="0 0 0" rpy="0 0 0" /> -->
+        <origin xyz="0.043 0 -0.12" rpy="0 0 0" />
         <geometry>
-          <mesh filename="package://pal_wsg_gripper_description/meshes/gripper_finger_link_collision.dae" scale="1 1 1"/>
+          <!-- <mesh filename="package://pal_wsg_gripper_description/meshes/gripper_finger_link_collision.dae" scale="1 1 1"/> -->
+          <box size="0.022 0.03 0.07"/>
         </geometry>
       </collision>
@@ -96,7 +98,9 @@
       </visual>
       <collision>
-        <origin xyz="0 0 0" rpy="0 0 0" />
+        <!-- <origin xyz="0 0 0" rpy="0 0 0" /> -->
+        <origin xyz="-0.043 0 -0.12" rpy="0 0 0" />
         <geometry>
-          <mesh filename="package://pal_wsg_gripper_description/meshes/gripper_finger_link_collision.dae" scale="-1 -1 1"/>
+          <!-- <mesh filename="package://pal_wsg_gripper_description/meshes/gripper_finger_link_collision.dae" scale="-1 -1 1"/> -->
+          <box size="0.022 0.03 0.07"/>
         </geometry>
       </collision>

Commit message: fix joint limit

File: pal_wsg_gripper_description/urdf/gripper.urdf.xacro (robot description, xacro)
@@ -6,5 +6,5 @@
   <xacro:include filename="$(find pal_wsg_gripper_description)/urdf/gripper.gazebo.xacro" />
   <xacro:property name="lower" value="0.0" />
-  <xacro:property name="upper" value="0.034" />
+  <xacro:property name="upper" value="0.068" />
   <xacro:property name="gripper_eps" value="0.001" />
   <xacro:macro name="pal_wsg_gripper" params="name parent *origin">

Commit message: fix reduction and limits

File: pal_wsg_gripper_description/urdf/gripper.urdf.xacro (robot description, xacro)
@@ -5,6 +5,6 @@
   <xacro:include filename="$(find pal_wsg_gripper_description)/urdf/gripper.transmission.xacro" />
   <xacro:include filename="$(find pal_wsg_gripper_description)/urdf/gripper.gazebo.xacro" />
-  <xacro:property name="lower" value="0.0" />
-  <xacro:property name="upper" value="0.068" />
+  <xacro:property name="lower" value="0.002" />
+  <xacro:property name="upper" value="0.034" />
   <xacro:property name="gripper_eps" value="0.001" />
   <xacro:macro name="pal_wsg_gripper" params="name parent *origin">
@@ -134,5 +134,5 @@
     </link>
     <xacro:parallel_fingers_joint joint_name_to_mimic="${name}_finger" virtual_joint_name="${name}_right_finger" />
-    <xacro:gripper_simple_transmission name="${name}" reduction="1.0"/>
+    <xacro:gripper_simple_transmission name="${name}" reduction="2.0"/>
   </xacro:macro>
 </robot>

Commit message: set eps to 0

File: pal_wsg_gripper_description/urdf/gripper.urdf.xacro (robot description, xacro)
@@ -7,5 +7,5 @@
   <xacro:property name="lower" value="0.002" />
   <xacro:property name="upper" value="0.034" />
-  <xacro:property name="gripper_eps" value="0.001" />
+  <xacro:property name="gripper_eps" value="0.000" />
   <xacro:macro name="pal_wsg_gripper" params="name parent *origin">
     <link name="${name}_link">

Commit message: Add gripper_tool_link

File: pal_wsg_gripper_description/urdf/gripper.urdf.xacro (robot description, xacro)
@@ -9,4 +9,20 @@
   <xacro:property name="gripper_eps" value="0.000" />
   <xacro:macro name="pal_wsg_gripper" params="name parent *origin">
+  <!-- Tool Link -->
+    <link name="${name}_tool_link">
+      <inertial>
+        <origin xyz="0 0 0" rpy="0 0 0" />
+        <mass value="0.0001" />
+        <inertia ixx="0.00001" ixy="0.0" ixz="0.0"
+                 iyy="0.00001" iyz="0.0"
+                 izz="0.00001" />
+      </inertial>
+    </link>
+    <joint name="${name}_tool_joint" type="fixed">
+      <insert_block name="origin"/>
+      <parent link="${parent}" />
+      <child link="${name}_tool_link" />
+       <axis xyz="0 0 0" />
+    </joint>
     <link name="${name}_link">
       <inertial>
