Commit message: Fix xacro warning
Same as https://gitlab/robots/tiago_robot/-/merge_requests/44

File: pal_wsg_gripper_description/urdf/deg_to_rad.urdf.xacro (robot description, xacro)
@@ -1,3 +1,3 @@
 <robot xmlns:xacro="http://ros.org/wiki/xacro">
-	<property name="deg_to_rad" value="0.01745329251994329577" />
+	<xacro:property name="deg_to_rad" value="0.01745329251994329577" />
 </robot>
